File: beatProj/beatProj.sch (KiCad schematic (older format))
At the start: 28 parts, among them IC1 UC2844AD8, U1 4N27

Commit message: completed schematic
Parts:
- D72: value BYV26E_Diode -> MLL4148
Changed lines of the file:
@@
 P 2900 1850
 F 0 "D72" V 2854 1978 50  0000 L CNN
-F 1 "BYV26E_Diode" V 2945 1978 50  0000 L CNN
+F 1 "MLL4148" V 2945 1978 50  0000 L CNN
 F 2 "" H 2900 1850 50  0001 C CNN
 F 3 "~" H 2900 1850 50  0001 C CNN
