File: beatProj/sheet2.sch (KiCad schematic (older format))
At the start: 25 parts

Commit message: completed schematic
Parts:
- added F3: 5A, 600V, ATM-5/KLK-5, symbol beatComponentLib:Fuseholder
- C40: renamed from C?; value CP1 -> 1mF 35V
- C42: renamed from C?; value C -> 10uF SMD
- D18: renamed from D?; value BYV26E_Diode -> ES3D
- DS3: renamed from D?; value LED -> Clear Green
- gave numbers to parts that had none: 1
Connections:
- net +24V: now also C40.2
- net RTN_OSC: now also C40.1, F3.2, F3.4
- new net -BAT: F3.1, F3.3
Changed lines of the file:
@@
 	6500 1700 6500 1900
 $Comp
-L beatComponentLib:IRFBE30PBF U?
+L beatComponentLib:IRFBE30PBF Q1
 U 1 1 5EF12270
 P 6200 3500
-F 0 "U?" H 6630 3553 60  0000 L CNN
+F 0 "Q1" H 6630 3553 60  0000 L CNN
 F 1 "IRFBE30PBF" H 6630 3447 60  0000 L CNN
 F 2 "TO220AB_VIS" H 6650 3240 60  0001 C CNN
@@
 $EndComp
 $Comp
-L beatComponentLib:LED D?
+L beatComponentLib:LED DS3
 U 1 1 5EF49451
 P 2300 6600
-F 0 "D?" V 2339 6483 50  0000 R CNN
-F 1 "LED" V 2248 6483 50  0000 R CNN
+F 0 "DS3" V 2339 6483 50  0000 R CNN
+F 1 "Clear Green" V 2248 6483 50  0000 R CNN
 F 2 "" H 2300 6600 50  0001 C CNN
 F 3 "~" H 2300 6600 50  0001 C CNN
@@
 $EndComp
 $Comp
-L beatComponentLib:C C?
+L beatComponentLib:C C42
 U 1 1 5EF49923
 P 3050 6800
-F 0 "C?" H 3165 6846 50  0000 L CNN
-F 1 "C" H 3165 6755 50  0000 L CNN
+F 0 "C42" H 3165 6846 50  0000 L CNN
+F 1 "10uF SMD" H 3165 6755 50  0000 L CNN
 F 2 "" H 3088 6650 50  0001 C CNN
 F 3 "~" H 3050 6800 50  0001 C CNN
@@
 $EndComp
 $Comp
-L beatComponentLib:CP1 C?
+L beatComponentLib:CP1 C40
 U 1 1 5EF49D1D
 P 4600 6800
-F 0 "C?" H 4715 6846 50  0000 L CNN
-F 1 "CP1" H 4715 6755 50  0000 L CNN
+F 0 "C40" H 4715 6846 50  0000 L CNN
+F 1 "1mF 35V" H 4715 6755 50  0000 L CNN
 F 2 "" H 4600 6800 50  0001 C CNN
 F 3 "~" H 4600 6800 50  0001 C CNN
@@
 $EndComp
 $Comp
-L beatComponentLib:BYV26E_Diode D?
+L beatComponentLib:BYV26E_Diode D18
 U 1 1 5EF4A0F7
 P 5750 7350
-F 0 "D?" H 5772 7600 50  0000 C CNN
-F 1 "BYV26E_Diode" H 5772 7516 40  0000 C CNN
+F 0 "D18" H 5772 7600 50  0000 C CNN
+F 1 "ES3D" H 5772 7516 40  0000 C CNN
 F 2 "" H 5750 7350 50  0001 C CNN
 F 3 "~" H 5750 7350 50  0001 C CNN
@@
 	6550 7350 5950 7350
 Wire Wire Line
-	5550 7350 3050 7350
+	5550 7350 4600 7350
 Connection ~ 1650 7350
 Wire Wire Line
@@
 Connection ~ 3050 7350
 Wire Wire Line
-	3050 7350 2300 7350
-Wire Wire Line
 	3050 6650 3050 6300
 Connection ~ 3050 6300
 Wire Wire Line
-	3050 6300 6500 6300
+	3050 6300 3800 6300
 Wire Wire Line
 	2300 6450 2300 6300
@@
 Wire Wire Line
 	6000 4300 6500 4300
+Wire Wire Line
+	4600 6650 4600 6300
+Connection ~ 4600 6300
+Wire Wire Line
+	4600 6300 6500 6300
+Wire Wire Line
+	4600 6950 4600 7350
+Connection ~ 4600 7350
+Wire Wire Line
+	4600 7350 3050 7350
+$Comp
+L beatComponentLib:Fuseholder F3
+U 1 1 5EF4B969
+P 2600 7700
+F 0 "F3" H 2600 7975 50  0000 C CNN
+F 1 "5A, 600V, ATM-5/KLK-5" H 2600 7884 50  0000 C CNN
+F 2 "" H 2600 7850 50  0001 C CNN
+F 3 "" H 2600 7850 50  0001 C CNN
+	1    2600 7700
+	1    0    0    -1
+$EndComp
+Wire Wire Line
+	3800 7650 2850 7650
+Connection ~ 3800 6300
+Wire Wire Line
+	3800 6300 4600 6300
+Wire Wire Line
+	2800 7750 2850 7750
+Wire Wire Line
+	2850 7750 2850 7650
+Connection ~ 2850 7650
+Wire Wire Line
+	2850 7650 2800 7650
+Text Label 2100 7650 2    50   ~ 0
+-BAT
+Wire Wire Line
+	2400 7650 2350 7650
+Wire Wire Line
+	2400 7750 2350 7750
+Wire Wire Line
+	2350 7750 2350 7650
+Connection ~ 2350 7650
+Wire Wire Line
+	2350 7650 2100 7650
+Wire Wire Line
+	3050 7350 2300 7350
+Wire Wire Line
+	3800 6300 3800 7650
 $EndSCHEMATC
